Commit message: Change controll parameters

File: controller/ros_controller.urdf.xacro (robot description, xacro)
@@ -4,8 +4,5 @@
        xmlns:interface="http://playerstage.sourceforge.net/gazebo/xmlschema/#interface">
   <gazebo>
-    <plugin name="gazebo_ros_controller" filename="libgazebo_ros_control.so">
-        <robotSimType>gazebo_ros_control/DefaultRobotHWSim</robotSimType>
-        <legacyModeNS>true</legacyModeNS>
-    </plugin>
+    <plugin name="gazebo_ros_controller" filename="libgazebo_ros_control.so" />
   </gazebo>
 </robot>

File: robots/youbot.urdf.xacro (robot description, xacro)
@@ -42,5 +42,5 @@
   </xacro:youbot_gripper>
   <!-- base laser front -->
-  <xacro:hokuyo_urg04_laser name="base_laser_front" parent="base" ros_topic="scan_front" update_rate="10" min_angle="-1.57" max_angle="1.57">
+  <xacro:hokuyo_urg04_laser name="base_laser_front" parent="base" ros_topic="scan_front" update_rate="100" min_angle="-1.57" max_angle="1.57">
     <origin xyz="0.3 0 -0.03" rpy="0 0 0"/>
   </xacro:hokuyo_urg04_laser>

File: urdf/youbot_arm/arm.urdf.xacro (robot description, xacro)
@@ -44,5 +44,5 @@
 			<axis xyz="0 0 -1"/>
 			<!--<calibration rising="${arm_1_ref}" falling="${arm_1_ref}"/>-->
-			<dynamics damping="1" friction="0.5" />
+			<dynamics damping="1" friction="1" />
 			<!-- damping - N*s/m, N*s*m/rad -->
 			<!-- friction - N, N*m -->
@@ -83,5 +83,5 @@
 			<axis xyz="0 1 0"/>
 			<!--<calibration rising="${arm_2_ref}" falling="${arm_2_ref}"/>-->
-			<dynamics damping="1" friction="0.5" />
+			<dynamics damping="1" friction="1" />
 			<limit effort="${9.5}" velocity="${M_PI / 2.0}" lower="0" upper="${joint_2_limit}"/>
       <!--safety_controller k_position="20" k_velocity="${2*9.5/M_PI}" soft_lower_limit="${threshold}" soft_upper_limit="${joint_2_limit_soft}" /-->
@@ -122,5 +122,5 @@
 			<child link="${name}_link_3"/>
 			<axis xyz="0 1 0"/>
-			<dynamics damping="1" friction="0.5" />
+			<dynamics damping="1" friction="1" />
 			<limit effort="${6.0}" velocity="${M_PI / 2.0}" lower="-${joint_3_limit}" upper="0"/>
       <!--safety_controller k_position="20" k_velocity="50" soft_lower_limit="-${joint_3_limit_soft}" soft_upper_limit="-${threshold}" /-->
@@ -154,5 +154,5 @@
 			<axis xyz="0 1 0" />
 			<!--<calibration rising="${arm_4_ref}" falling="${arm_4_ref}"/>-->
-			<dynamics damping="1" friction="0.5" />
+			<dynamics damping="1" friction="1" />
 			<limit effort="${2.0}" velocity="${M_PI / 2.0}" lower="0" upper="${joint_4_limit}"/>
 			<!--safety_controller k_position="20" k_velocity="100" soft_lower_limit="0" soft_upper_limit="${joint_4_limit_soft}" /-->
@@ -186,5 +186,5 @@
 			<axis xyz="0 0 -1" />
 			<!--<calibration rising="${arm_5_ref}" falling="${arm_5_ref}"/>-->
-			<dynamics damping="0.5" friction="0.5" />
+			<dynamics damping="1" friction="1" />
 			<limit effort="${1.0}" velocity="${M_PI / 2.0}" lower="0" upper="${joint_5_limit}" />
       <!--safety_controller k_position="20" k_velocity="100" soft_lower_limit="0" soft_upper_limit="${joint_5_limit_soft}" /-->
